File: design/switchbox/switchbox.kicad_pcb (KiCad board)
At the start: 2 copper layers, 70 x 32 mm, 7 parts, among them J1 A0, J2 GND, SW1 SW1, SW2 SW2

Commit message: Added label to PCB
Other:
- board text added: "beetchef"
- board text added: "switchbox"
Changed lines of the file:
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@@
   (general
     (thickness 1.6)
-    (drawings 12)
+    (drawings 14)
     (tracks 26)
     (zones 0)
@@
     (47 F.CrtYd user hide)
     (48 B.Fab user)
-    (49 F.Fab user hide)
+    (49 F.Fab user)
   )
   (setup
@@
     )
   )
+  (gr_text switchbox (at 189.23 55.88) (layer F.Fab)
+    (effects (font (size 2 2.5) (thickness 0.2)) (justify left))
+  )
+  (gr_text beetchef (at 189.23 53.34) (layer F.Fab)
+    (effects (font (size 2 2.5) (thickness 0.3)) (justify left))
+  )
   (gr_line (start 156.06 49.28) (end 156.06 59.28) (layer Edge.Cuts) (width 0.05))

Commit message: Changed label for analog pin terminal
Parts:
- J1: value A0 -> +5V
Changed lines of the file:
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@@
       (effects (font (size 1 1) (thickness 0.15)))
     )
-    (fp_text value A0 (at 2.54 0) (layer F.Fab)
+    (fp_text value +5V (at 3.175 0) (layer F.Fab)
       (effects (font (size 1 1) (thickness 0.15)))
     )
